Commit message: NEW：服务器编写完成

File: ARV_V1_MODEL/urdf/ARV_V1_MODEL.urdf (robot description, URDF)
Before this commit: robot ARV_V1_MODEL, 7 links, 6 joints
Links:
- added link world
Joints:
- added joint world_fixed: type fixed, parent world, child base_link, origin xyz=0 0 0.5 rpy=0 0 0

File: ARV_V1_MOVEIT/config/ARV_V1_MODEL.ros2_control.xacro (robot description, xacro)
@@ -5,9 +5,10 @@
         <ros2_control name="${name}" type="system">
             <hardware>
-                <!-- By default, set up controllers for simulation. This won't work on real hardware -->
+                <!-- 使用 mock 硬件用于测试和开发 -->
                 <plugin>mock_components/GenericSystem</plugin>
             </hardware>
             <joint name="joint_1">
                 <command_interface name="position"/>
+                <command_interface name="effort"/>  <!-- 添加力矩命令接口 -->
                 <state_interface name="position">
                   <param name="initial_value">${initial_positions['joint_1']}</param>
@@ -18,4 +19,5 @@
             <joint name="joint_2">
                 <command_interface name="position"/>
+                <command_interface name="effort"/>  <!-- 添加力矩命令接口 -->
                 <state_interface name="position">
                   <param name="initial_value">${initial_positions['joint_2']}</param>
@@ -26,4 +28,5 @@
             <joint name="joint_3">
                 <command_interface name="position"/>
+                <command_interface name="effort"/>  <!-- 添加力矩命令接口 -->
                 <state_interface name="position">
                   <param name="initial_value">${initial_positions['joint_3']}</param>
@@ -34,4 +37,5 @@
             <joint name="joint_4">
                 <command_interface name="position"/>
+                <command_interface name="effort"/>  <!-- 添加力矩命令接口 -->
                 <state_interface name="position">
                   <param name="initial_value">${initial_positions['joint_4']}</param>
@@ -42,4 +46,5 @@
             <joint name="joint_5">
                 <command_interface name="position"/>
+                <command_interface name="effort"/>  <!-- 添加力矩命令接口 -->
                 <state_interface name="position">
                   <param name="initial_value">${initial_positions['joint_5']}</param>
@@ -50,4 +55,5 @@
             <joint name="joint_6">
                 <command_interface name="position"/>
+                <command_interface name="effort"/>  <!-- 添加力矩命令接口 -->
                 <state_interface name="position">
                   <param name="initial_value">${initial_positions['joint_6']}</param>

File: ARV_V1_MOVEIT/config/ARV_V1_MODEL.urdf.xacro (robot description, xacro)
@@ -6,4 +6,5 @@
     <!-- Import control_xacro -->
     <xacro:include filename="ARV_V1_MODEL.ros2_control.xacro" />
+    <!-- ros2_control 标签（使用 mock 硬件） -->
     <xacro:ARV_V1_MODEL_ros2_control name="FakeSystem" initial_positions_file="$(arg initial_positions_file)"/>
 </robot>
