Commit message: NEW：仿真复现成功

File: ARV_V1_MODEL/urdf/.mujoco_temp.urdf (robot description, URDF)
Before this commit: robot ARV_V1_MODEL, 8 links, 7 joints
Links:
- link base_link: geometry collision mesh filename=base_link.STL; visual mesh filename=base_link.STL
- link link1_double8009: geometry collision mesh filename=link1_double8009.STL; visual mesh filename=link1_double8009.STL
- link link2_arm1: geometry collision mesh filename=link2_arm1.STL; visual mesh filename=link2_arm1.STL
- link link3_sight: geometry collision mesh filename=link3_sight.STL; visual mesh filename=link3_sight.STL
- link link4_arm2: geometry collision mesh filename=link4_arm2.STL; visual mesh filename=link4_arm2.STL
- link link5_4310pitch: geometry collision mesh filename=link5_4310pitch.STL; visual mesh filename=link5_4310pitch.STL
- link link6_2006roll: geometry collision mesh filename=link6_2006roll.STL; visual mesh filename=link6_2006roll.STL

Commit message: new：shit

File: ARV_V1_MODEL/urdf/.mujoco_temp.urdf (robot description, URDF)
Before this commit: robot ARV_V1_MODEL, 8 links, 7 joints
Joints:
- joint joint_1: origin xyz=0 0 0 rpy=1.5708 0 0 -> xyz=0 0 0 rpy=0 0 0

Commit message: FUNNY TIME: v1

File: ARV_V1_MODEL/urdf/.mujoco_temp.urdf (robot description, URDF)
Before this commit: robot ARV_V1_MODEL, 8 links, 7 joints
Joints:
- joint joint_1: axis 0 1 0 -> 0 0 1

File: ARV_V1_MODEL/urdf/ARV_V1_MODEL.urdf (robot description, URDF)
Before this commit: robot ARV_V1_MODEL, 8 links, 7 joints
Joints:
- joint joint_1: axis 0 1 0 -> 0 0 1; origin xyz=0 0 0 rpy=1.5708 0 0 -> xyz=0 0 0 rpy=0 0 0

Commit message: 测试用修改惯量（不确定

File: ARV_V1_MODEL/urdf/.mujoco_temp.urdf (robot description, URDF)
Before this commit: robot ARV_V1_MODEL, 8 links, 7 joints
Joints:
- joint joint_2: origin xyz=0 0 0 rpy=0 0 0 -> xyz=0 0 0 rpy=1.5708 0 0

File: ARV_V1_MODEL/urdf/ARV_V1_MODEL.urdf (robot description, URDF)
Before this commit: robot ARV_V1_MODEL, 8 links, 7 joints
Joints:
- joint joint_2: origin xyz=0 0 0 rpy=0 0 0 -> xyz=0 0 0 rpy=1.5708 0 0
