Commit message: ENH: 场景模型搭建demo调试完成

File: arv_v1_model/urdf/arv_v1_model.urdf (robot description, URDF)
Before this commit: robot arv_v1_model, 8 links, 7 joints
Joints:
- joint world_fixed: origin xyz=0 0 0.5 rpy=0 0 0 -> xyz=0 0 0.35 rpy=0 0 0

File: arv_v1_model/urdf/obstacles/energy_core.urdf (robot description, URDF)
Before this commit: robot energy_core, 1 links, 0 joints
Links:
- link base_link: geometry collision mesh filename=package://arv_v1_model/meshes/obstacles/energy_core.STL; visual mesh filename=package://arv_v1_model/meshes/obstacles/energy_core.STL
