Commit message: enh：新urdf

File: arv_v1_model/urdf/arv_v1_old.urdf (robot description, URDF)
Before this commit: robot arv_v1, 11 links, 10 joints
Joints:
- joint joint_2: origin xyz=0 0 0.055 rpy=1.5707963267949 0 0 -> xyz=0.03215 0 0.131 rpy=1.5707963267949 0 0
- joint joint_3: origin xyz=0.440 0 0 rpy=0 0 0 -> xyz=0.381000000000038 0 0 rpy=0 0 0
- joint joint_5: origin xyz=0 0 0.3505 rpy=-1.5707963267949 0 0 -> xyz=0.00129999999995989 -0.00719999999941014 0.43888820457198 rpy=-1.5707963267949 0 0
