Commit message: 向后兼容的包名

File: arv_v1_model/urdf/arv_v1.urdf (robot description, URDF)
Before this commit: robot arv_v2, 9 links, 8 joints
Links:
- link base_link: geometry collision mesh filename=package://arv_v1_model/meshes/base_link.STL; visual mesh filename=package://arv_v1_model/meshes/base_link.STL
- link link1: geometry collision mesh filename=package://arv_v1_model/meshes/link1.STL; visual mesh filename=package://arv_v1_model/meshes/link1.STL
- link link2: geometry collision mesh filename=package://arv_v1_model/meshes/link2.STL; visual mesh filename=package://arv_v1_model/meshes/link2.STL
- link link3: geometry collision mesh filename=package://arv_v1_model/meshes/link3.STL; visual mesh filename=package://arv_v1_model/meshes/link3.STL
- link link4: geometry collision mesh filename=package://arv_v1_model/meshes/link4.STL; visual mesh filename=package://arv_v1_model/meshes/link4.STL
- link link5: geometry collision mesh filename=package://arv_v1_model/meshes/link5.STL; visual mesh filename=package://arv_v1_model/meshes/link5.STL
- link link6: geometry collision mesh filename=package://arv_v1_model/meshes/link6.STL; visual mesh filename=package://arv_v1_model/meshes/link6.STL
- link link_gripper1: geometry collision mesh filename=package://arv_v1_model/meshes/link_gripper1.STL; visual mesh filename=package://arv_v1_model/meshes/link_gripper1.STL
- link link_gripper2: geometry collision mesh filename=package://arv_v1_model/meshes/link_gripper2.STL; visual mesh filename=package://arv_v1_model/meshes/link_gripper2.STL

Commit message: fix1

File: arv_v1_model/urdf/arv_v1.urdf (robot description, URDF)
Before this commit: robot arv_v1, 9 links, 8 joints
Joints:
- removed joint joint1
- removed joint joint2
- removed joint joint3
- removed joint joint4
- removed joint joint5
- removed joint joint6
- added joint joint_1: type revolute, parent base_link, child link1, origin xyz=0 0 0 rpy=0 0 0, axis 0 0 1, limit lower=-3.2 upper=3.2 effort=40 velocity=20
- added joint joint_2: type revolute, parent link1, child link2, origin xyz=0.03215 0 0.131 rpy=1.5707963267949 0 0, axis 0 0 1, limit lower=-3.2 upper=3.2 effort=40 velocity=20
- added joint joint_3: type revolute, parent link2, child link3, origin xyz=0.381000000000038 0 0 rpy=0 0 0, axis 0 0 -1, limit lower=-3.2 upper=3.2 effort=40 velocity=20
- added joint joint_4: type revolute, parent link3, child link4, origin xyz=0 0 0 rpy=1.5707963267949 0 0, axis 0 0 1, limit lower=-3.2 upper=3.2 effort=1.2 velocity=40
- added joint joint_5: type revolute, parent link4, child link5, origin xyz=0.00129999999995989 -0.00719999999941014 0.43888820457198 rpy=-1.5707963267949 0 0, axis 0 0 -1, limit lower=-3.2 upper=3.2 effort=7 velocity=20
- added joint joint_6: type revolute, parent link5, child link6, origin xyz=0 0 0 rpy=1.57079632679552 0 0, axis 0 0 1, limit lower=-3.2 upper=3.2 effort=1 velocity=20
- joint joint_gripper1: limit lower=0 upper=0.04 effort=7 velocity=0 -> lower=0 upper=0.04 effort=7 velocity=0.1
- joint joint_gripper2: limit lower=-0.04 upper=0 effort=7 velocity=0 -> lower=-0.04 upper=0 effort=7 velocity=0.1

File: arv_v1_moveit/config/arv_v1_model.ros2_control.xacro (robot description, xacro)
@@ -62,4 +62,15 @@
                 <state_interface name="effort"/>
             </joint>
+            <!-- 夹爪主动关节 -->
+            <joint name="joint_gripper1">
+                <command_interface name="position"/>
+                <command_interface name="effort"/>  <!-- 添加力矩命令接口 -->
+                <state_interface name="position">
+                  <param name="initial_value">${initial_positions['joint_gripper1']}</param>
+                </state_interface>
+                <state_interface name="velocity"/>
+                <state_interface name="effort"/>
+            </joint>
+            <!-- joint_gripper2 是 mimic 关节，由 robot_state_publisher 自动计算，不加 ros2_control 接口 -->
         </ros2_control>
     </xacro:macro>

File: arv_v1_moveit/config/arv_v1_model.urdf.xacro (robot description, xacro)
@@ -2,6 +2,6 @@
 <robot xmlns:xacro="http://www.ros.org/wiki/xacro" name="arv_v1_model">
     <xacro:arg name="initial_positions_file" default="initial_positions.yaml" />
-    <!-- Import arv_v1_model urdf file -->
-    <xacro:include filename="$(find arv_v1_model)/urdf/arv_v1_model.urdf" />
+    <!-- Import arv_v1 urdf file -->
+    <xacro:include filename="$(find arv_v1_model)/urdf/arv_v1.urdf" />
     <!-- Import control_xacro -->
     <xacro:include filename="arv_v1_model.ros2_control.xacro" />

Commit message: fix: 修复被错误回溯的urdf

File: arv_v1_model/urdf/arv_v1.urdf (robot description, URDF)
Before this commit: robot arv_v1, 9 links, 8 joints
Links:
- added link tcp
Joints:
- added joint joint_tcp: type fixed, parent link6, child tcp, origin xyz=0 0.000 0.179 rpy=0 0 0, axis 0 0 0

Commit message: ENH: 完成完整迁移层，修复虚拟joint

File: arv_v1_model/urdf/arv_v1.urdf (robot description, URDF)
Before this commit: robot arv_v1, 10 links, 9 joints
Links:
- added link world
Joints:
- added joint world_fixed: type fixed, parent world, child base_link, origin xyz=0 0 0.35 rpy=0 0 0

Commit message: 1

File: arv_v1_model/urdf/arv_v1.urdf (robot description, URDF)
Before this commit: robot arv_v1, 11 links, 10 joints
Joints:
- joint world_fixed: origin xyz=0 0 0.35 rpy=0 0 0 -> xyz=-0.1 0 0.15 rpy=0 0 0

Commit message: fix：修复惯量问题

File: arv_v1_model/urdf/arv_v1.urdf (robot description, URDF)
Before this commit: robot arv_v1, 11 links, 10 joints
Links:
- link base_link: mass 0.349525984991482 -> 0.980
- link link1: mass 1.22525961510696 -> 2.485
- link link3: mass 1.11704493186519 -> 1.612
- link link4: mass 0.568849364384239 -> 1.021
- link link5: mass 0.100227688220142 -> 0.180
- link link6: mass 0.0590335082391964 -> 0.106
- link link_gripper1: mass 0.0581710450017314 -> 0.104
- link link_gripper2: mass 0.0581710450017313 -> 0.104

Commit message: cherry-pick: 58305c6 refactor(服务框架+serial+笛卡尔修复, mujoco保留ours)

File: arv_v1_model/urdf/arv_v1.urdf (robot description, URDF)
Before this commit: robot arv_v1, 11 links, 10 joints
Joints:
- joint joint_gripper1: limit lower=0 upper=0.04 effort=7 velocity=0.1 -> lower=0 upper=0.04 effort=70 velocity=0.1
- joint joint_gripper2: limit lower=-0.04 upper=0 effort=7 velocity=0.1 -> lower=-0.04 upper=0 effort=70 velocity=0.1

Commit message: fix: 修复无限制的限位

File: arv_v1_model/urdf/arv_v1.urdf (robot description, URDF)
Before this commit: robot arv_v1, 11 links, 10 joints
Links:
- link base_link: geometry collision cylinder length=0.06 radius=0.06; visual mesh filename=package://arv_v1_model/meshes/base_link.STL
- link link1: geometry collision cylinder length=0.12 radius=0.04; visual mesh filename=package://arv_v1_model/meshes/link1.STL
- link link2: geometry collision cylinder length=0.36 radius=0.025; visual mesh filename=package://arv_v1_model/meshes/link2.STL
- link link3: geometry collision cylinder length=0.06 radius=0.03; visual mesh filename=package://arv_v1_model/meshes/link3.STL
- link link4: geometry collision cylinder length=0.43 radius=0.02; visual mesh filename=package://arv_v1_model/meshes/link4.STL
- link link5: geometry collision cylinder length=0.03 radius=0.015; visual mesh filename=package://arv_v1_model/meshes/link5.STL
- link link6: geometry collision cylinder length=0.17 radius=0.015; visual mesh filename=package://arv_v1_model/meshes/link6.STL
- link link_gripper1: geometry collision box size=0.012 0.012 0.06; visual mesh filename=package://arv_v1_model/meshes/link_gripper1.STL
- link link_gripper2: geometry collision box size=0.012 0.012 0.06; visual mesh filename=package://arv_v1_model/meshes/link_gripper2.STL
Joints:
- joint joint_1: limit lower=-3.2 upper=3.2 effort=40 velocity=20 -> lower=-1.13 upper=1.13 effort=40 velocity=20
- joint joint_2: limit lower=-3.2 upper=3.2 effort=40 velocity=20 -> lower=0.44 upper=2.88 effort=40 velocity=20
- joint joint_3: limit lower=-3.2 upper=3.2 effort=40 velocity=20 -> lower=-1.48 upper=3.05 effort=40 velocity=20
- joint joint_4: limit lower=-3.2 upper=3.2 effort=1.2 velocity=40 -> lower=-3.05 upper=3.05 effort=1.2 velocity=40
- joint joint_5: limit lower=-3.2 upper=3.2 effort=7 velocity=20 -> lower=-1.48 upper=1.48 effort=7 velocity=20
- joint joint_6: limit lower=-3.2 upper=3.2 effort=1 velocity=20 -> effort=1 velocity=20; type revolute -> continuous

Commit message: fix：修复夹爪长度过长问题

File: arv_v1_model/urdf/arv_v1.urdf (robot description, URDF)
Before this commit: robot arv_v1, 11 links, 10 joints
Links:
- link link6: geometry collision cylinder length=0.06 radius=0.015; visual mesh filename=package://arv_v1_model/meshes/link6.STL

Commit message: FIX:修复真实电机扭矩

File: arv_v1_model/urdf/arv_v1.urdf (robot description, URDF)
Before this commit: robot arv_v1, 11 links, 10 joints
Joints:
- joint joint_1: limit lower=-1.2217 upper=1.2217 effort=40 velocity=20 -> lower=-1.2217 upper=1.2217 effort=27 velocity=20
- joint joint_3: limit lower=-1.5708 upper=3.1416 effort=40 velocity=20 -> lower=-1.5708 upper=3.1416 effort=27 velocity=20

Commit message: ENH: enhance torque of joint and packages problem

File: arv_v1_model/urdf/arv_v1.urdf (robot description, URDF)
Before this commit: robot arv_v1, 11 links, 10 joints
Joints:
- joint joint_3: limit lower=-1.5708 upper=3.1416 effort=27 velocity=20 -> lower=-1.5708 upper=3.1416 effort=54 velocity=10

Commit message: ENH: 下位机静态参数标定完成

File: arv_v1_model/urdf/arv_v1.urdf (robot description, URDF)
Before this commit: robot arv_v1, 11 links, 10 joints
Links:
- link link3: mass 1.612 -> 3.485

Commit message: ENH:同步下位机标定质量惯量

File: arv_v1_model/urdf/arv_v1.urdf (robot description, URDF)
Before this commit: robot arv_v1, 11 links, 10 joints
Links:
- link link3: mass 3.485 -> 2.211
- link link4: mass 1.021 -> 2.295

Commit message: fix：修复反轴&pid行为

File: arv_v1_model/urdf/arv_v1.urdf (robot description, URDF)
Before this commit: robot arv_v1, 11 links, 10 joints
Joints:
- joint joint_5: axis 0 0 -1 -> 0 0 1

Commit message: ENH: 同步限位

File: arv_v1_model/urdf/arv_v1.urdf (robot description, URDF)
Before this commit: robot arv_v1, 11 links, 10 joints
Joints:
- joint joint_4: limit lower=-3.1416 upper=3.1416 effort=1.2 velocity=40 -> lower=-2.975 upper=3.14 effort=1.2 velocity=40

Commit message: ENH：同步限位，添加注入脚本

File: arv_v1_model/urdf/arv_v1.urdf (robot description, URDF)
Before this commit: robot arv_v1, 11 links, 10 joints
Joints:
- joint joint_2: limit lower=0.5236 upper=2.9671 effort=40 velocity=20 -> lower=0.49 upper=3.14 effort=40 velocity=20
- joint joint_3: limit lower=-1.5708 upper=3.1416 effort=54 velocity=10 -> lower=-0.90 upper=0.70 effort=54 velocity=10

Commit message: ENH: 标定质量结束 :# 请为您的变更输入提交说明。以 '#' 开始的行将被忽略，而一个空的提交

File: arv_v1_model/urdf/arv_v1.urdf (robot description, URDF)
Before this commit: robot arv_v1, 11 links, 10 joints
Links:
- link link2: mass 1.13036010199932 -> 3.087; geometry collision cylinder length=0.44 radius=0.025; visual mesh filename=package://arv_v1_model/meshes/link2.STL
- link link3: mass 2.211 -> 1.270
- link link4: mass 2.295 -> 0.724; geometry collision cylinder length=0.35 radius=0.02; visual mesh filename=package://arv_v1_model/meshes/link4.STL
- link link6: mass 0.106 -> 0.706
Joints:
- joint joint_2: origin xyz=0.03215 0 0.131 rpy=1.5707963267949 0 0 -> xyz=0 0 0.055 rpy=1.5707963267949 0 0
- joint joint_3: origin xyz=0.381000000000038 0 0 rpy=0 0 0 -> xyz=0.440 0 0 rpy=0 0 0
- joint joint_5: origin xyz=0.00129999999995989 -0.00719999999941014 0.43888820457198 rpy=-1.5707963267949 0 0 -> xyz=0 0 0.3505 rpy=-1.5707963267949 0 0

File: arv_v1_model/urdf/arv_v1_new.urdf (robot description, URDF)
Before this commit: robot arv_v1, 11 links, 10 joints
Links:
- link link2: mass 1.13036010199932 -> 3.087
- link link3: mass 2.211 -> 1.270
- link link4: mass 2.295 -> 0.724
- link link6: mass 0.106 -> 0.706
