Commit message: fix: 修正关节限位弧度换算误差
deg→rad 精确换算 (之前截断导致 ~5° 偏差):
  J1 ±70° → ±1.2217, J2 30°~170° → 0.5236~2.9671,
  J3 -90°~180° → -1.5708~3.1416, J4 ±180° → ±3.1416,
  J5 ±90° → ±1.5708
三处同步: URDF, joint_limits.yaml, cartesian_controller IK clamp

Co-Authored-By: Claude Opus 4.6 (1M context) <noreply@anthropic.com>

File: arv_v1_model/urdf/arv_v1.urdf (robot description, URDF)
Before this commit: robot arv_v1, 11 links, 10 joints
Joints:
- joint joint_1: limit lower=-1.13 upper=1.13 effort=40 velocity=20 -> lower=-1.2217 upper=1.2217 effort=40 velocity=20
- joint joint_2: limit lower=0.44 upper=2.88 effort=40 velocity=20 -> lower=0.5236 upper=2.9671 effort=40 velocity=20
- joint joint_3: limit lower=-1.48 upper=3.05 effort=40 velocity=20 -> lower=-1.5708 upper=3.1416 effort=40 velocity=20
- joint joint_4: limit lower=-3.05 upper=3.05 effort=1.2 velocity=40 -> lower=-3.1416 upper=3.1416 effort=1.2 velocity=40
- joint joint_5: limit lower=-1.48 upper=1.48 effort=7 velocity=20 -> lower=-1.5708 upper=1.5708 effort=7 velocity=20

Commit message: enh: LIN 失败时诊断哪个关节超限
IK 失败时调 solveUnclamped() 获取无限位约束的最近解，
对比 kJointLower/Upper 报告具体哪个关节超了多少。
service response message 包含: 步数、插值比例、超限关节及其值。

Co-Authored-By: Claude Opus 4.6 (1M context) <noreply@anthropic.com>

File: arv_v1_model/urdf/arv_v1.urdf (robot description, URDF)
Before this commit: robot arv_v1, 11 links, 10 joints
Joints:
- joint world_fixed: origin xyz=-0.1 0 0.15 rpy=0 0 0 -> xyz=-0.05 0 0.15 rpy=0 0 0

Commit message: fix: Read Current 坐标系修正 — world frame → base_link frame
实测 Pitch1 轴线距地面 35cm, D1=5.5cm → base_link 离地 29.5cm。
URDF world_fixed z: 0.15 → 0.295, 同步 mujoco kWorldBaseOffset。

Co-Authored-By: Claude Opus 4.6 (1M context) <noreply@anthropic.com>

File: arv_v1_model/urdf/arv_v1.urdf (robot description, URDF)
Before this commit: robot arv_v1, 11 links, 10 joints
Joints:
- joint world_fixed: origin xyz=-0.05 0 0.15 rpy=0 0 0 -> xyz=-0.05 0 0.295 rpy=0 0 0
